File: som/pixieboard.kicad_sch (KiCad schematic)
At the start: 23 parts, among them J1 Conn_02x20_Counter_Clockwise, J2 Conn_02x20_Counter_Clockwise, J3 Conn_02x20_Counter_Clockwise, J4 Conn_02x20_Counter_Clockwise, J5 Conn_02x20_Counter_Clockwise, J6 Conn_02x20_Counter_Clockwise, SW1 SW_DIP_x03, U1 XC7A200T-3FBG484E, U4 W25Q128JVS

Commit message: GTP stuff
Parts:
- removed C57: 100nF, Capacitor_SMD:C_0402_1005Metric, symbol Device:C_Small
- removed R3, R4, R5: 10K, Resistor_SMD:R_0402_1005Metric_Pad0.72x0.64mm_HandSolder, symbol Device:R_Small
- removed SW1: SW_DIP_x03, Button_Switch_SMD:SW_DIP_SPSTx03_Slide_Omron_A6S-310x_W8.9mm_P2.54mm, symbol Switch:SW_DIP_x03
- removed U4: W25Q128JVS, Package_SO:SOIC-8_5.23x5.23mm_P1.27mm, symbol Memory_Flash:W25Q128JVS
Connections:
- net MGT_RX1+: now also J2.17 (Pin_17), J2.24 (Pin_24); no longer J2.11 (Pin_11), J2.30 (Pin_30)
- net MGT_RX1-: now also J2.18 (Pin_18), J2.23 (Pin_23); no longer J2.12 (Pin_12), J2.29 (Pin_29)
- net MGT_RX2+: now also J2.11 (Pin_11), J2.30 (Pin_30); no longer J2.14 (Pin_14), J2.27 (Pin_27)
- net MGT_RX2-: now also J2.12 (Pin_12), J2.29 (Pin_29); no longer J2.15 (Pin_15), J2.26 (Pin_26)
- net MGT_RX3+: now also J2.14 (Pin_14), J2.27 (Pin_27); no longer J2.17 (Pin_17), J2.24 (Pin_24)
- net MGT_RX3-: now also J2.15 (Pin_15), J2.26 (Pin_26); no longer J2.18 (Pin_18), J2.23 (Pin_23)
- net +1V2 renamed MTGAVTT
Other:
- moved on the sheet: J1, R19, U1H

Commit message: A little 155 pin I/O breakout
Parts:
- added J7: Conn_02x20_Counter_Clockwise, Mezzanine:YXT-BB10-40P-02, symbol Connector_Generic:Conn_02x20_Counter_Clockwise
Connections:
- net TDI_BANK0: now reaches U1.R13 (TDI_0)
- net TMS_BANK0: now reaches U1.T13 (TMS_0)
- net TDO_BANK0: now reaches U1.U13 (TDO_0)
- net TCK_BANK0: now reaches U1.V12 (TCK_0)
- net IO_AA9_BANK13: now reaches J6.1 (Pin_1)
- net IO_AA9_BANK13: now also U1.AA9 (IO_L8P_T1_13)
- net IO_W12_BANK13: now reaches J6.10 (Pin_10)
- net IO_W12_BANK13: now also U1.W12 (IO_L12N_T1_MRCC_13)
- net IO_V14_BANK13: now reaches J6.11 (Pin_11)
- net IO_V14_BANK13: now also U1.V14 (IO_L13N_T2_MRCC_13)
- net IO_V15_BANK13: now reaches J6.12 (Pin_12)
- net IO_V15_BANK13: now also U1.V15 (IO_L14N_T2_SRCC_13)
- net IO_W14_BANK13: now reaches J6.13 (Pin_13)
- net IO_W14_BANK13: now also U1.W14 (IO_L6P_T0_13)
- net IO_W15_BANK13: now reaches J6.14 (Pin_14)
- net IO_W15_BANK13: now also U1.W15 (IO_L16P_T2_13)
- net IO_T16_BANK13: now reaches J6.15 (Pin_15)
- net IO_T16_BANK13: now also U1.T16 (IO_L17P_T2_13)
- net IO_U16_BANK13: now reaches J6.16 (Pin_16)
- net IO_U16_BANK13: now also U1.U16 (IO_L17N_T2_13)
- net IO_W10_BANK13: now reaches J6.2 (Pin_2)
- net IO_W10_BANK13: now also U1.W10 (IO_L10N_T1_13)
- net IO_W16_BANK13: now reaches J6.21 (Pin_21)
- net IO_W16_BANK13: now also U1.W16 (IO_L16N_T2_13)
- net IO_Y17_BANK13: now reaches J6.22 (Pin_22)
- net IO_Y17_BANK13: now also U1.Y17 (IO_0_13)
- net IO_AB17_BANK13: now reaches J6.23 (Pin_23)
- net IO_AB17_BANK13: now also U1.AB17 (IO_L2N_T0_13)
- net IO_AA16_BANK13: now reaches J6.24 (Pin_24)
- net IO_AA16_BANK13: now also U1.AA16 (IO_L1N_T0_13)
- net IO_AB16_BANK13: now reaches J6.25 (Pin_25)
- net IO_AB16_BANK13: now also U1.AB16 (IO_L2P_T0_13)
- net IO_Y16_BANK13: now reaches J6.26 (Pin_26)
- net IO_Y16_BANK13: now also U1.Y16 (IO_L1P_T0_13)
- net IO_AA15_BANK13: now reaches J6.27 (Pin_27)
- net IO_AA15_BANK13: now also U1.AA15 (IO_L4P_T0_13)
- net IO_AB15_BANK13: now reaches J6.28 (Pin_28)
- net IO_AB15_BANK13: now also U1.AB15 (IO_L4N_T0_13)
- net IO_Y14_BANK13: now reaches J6.29 (Pin_29)
- net IO_Y14_BANK13: now also U1.Y14 (IO_L6N_T0_VREF_13)
- net IO_AA14_BANK13: now reaches J6.30 (Pin_30)
- net IO_AA14_BANK13: now also U1.AA14 (IO_L5N_T0_13)
- net IO_AB13_BANK13: now reaches J6.31 (Pin_31)
- net IO_AB13_BANK13: now also U1.AB13 (IO_L3N_T0_DQS_13)
- net IO_AA13_BANK13: now reaches J6.32 (Pin_32)
- net IO_AA13_BANK13: now also U1.AA13 (IO_L3P_T0_DQS_13)
- net IO_Y13_BANK13: now reaches J6.33 (Pin_33)
- net IO_Y13_BANK13: now also U1.Y13 (IO_L5P_T0_13)
- net IO_AB12_BANK13: now reaches J6.34 (Pin_34)
- net IO_AB12_BANK13: now also U1.AB12 (IO_L7N_T1_13)
- net IO_Y12_BANK13: now reaches J6.35 (Pin_35)
- net IO_Y12_BANK13: now also U1.Y12 (IO_L11N_T1_SRCC_13)
- net IO_Y11_BANK13: now reaches J6.36 (Pin_36)
- net IO_Y11_BANK13: now also U1.Y11 (IO_L11P_T1_SRCC_13)
- net IO_AB11_BANK13: now reaches J6.37 (Pin_37)
- net IO_AB11_BANK13: now also U1.AB11 (IO_L7P_T1_13)
- net IO_AA11_BANK13: now reaches J6.38 (Pin_38)
- net IO_AA11_BANK13: now also U1.AA11 (IO_L9N_T1_DQS_13)
- net IO_AA10_BANK13: now reaches J6.39 (Pin_39)
- net IO_AA10_BANK13: now also U1.AA10 (IO_L9P_T1_DQS_13)
- net IO_T14_BANK13: now reaches J6.4 (Pin_4)
- net IO_T14_BANK13: now also U1.T14 (IO_L15P_T2_DQS_13)
- net IO_AB10_BANK13: now reaches J6.40 (Pin_40)
- net IO_AB10_BANK13: now also U1.AB10 (IO_L8N_T1_13)
- net IO_V10_BANK13: now reaches J6.5 (Pin_5)
- net IO_V10_BANK13: now also U1.V10 (IO_L10P_T1_13)
- net IO_W11_BANK13: now reaches J6.6 (Pin_6)
- net IO_W11_BANK13: now also U1.W11 (IO_L12P_T1_MRCC_13)
- net IO_T15_BANK13: now reaches J6.7 (Pin_7)
- net IO_T15_BANK13: now also U1.T15 (IO_L15N_T2_DQS_13)
- net IO_U15_BANK13: now reaches J6.8 (Pin_8)
- net IO_U15_BANK13: now also U1.U15 (IO_L14P_T2_SRCC_13)
- net IO_V13_BANK13: now reaches J6.9 (Pin_9)
- net IO_V13_BANK13: now also U1.V13 (IO_L13P_T2_MRCC_13)
- net IO_M16_BANK15: now reaches J4.1 (Pin_1)
- net IO_M16_BANK15: now also U1.M16 (IO_L24N_T3_RS0_15)
- net IO_J16_BANK15: now reaches J4.10 (Pin_10)
- net IO_J16_BANK15: now also U1.J16 (IO_0_15)
- net IO_K18_BANK15: now reaches J4.11 (Pin_11)
- net IO_K18_BANK15: now also U1.K18 (IO_L13P_T2_MRCC_15)
- net IO_K17_BANK15: now reaches J4.12 (Pin_12)
- net IO_K17_BANK15: now also U1.K17 (IO_L21P_T3_DQS_15)
- net IO_J14_BANK15: now reaches J4.13 (Pin_13)
- net IO_J14_BANK15: now also U1.J14 (IO_L3P_T0_DQS_AD1P_15)
- net IO_H14_BANK15: now reaches J4.14 (Pin_14)
- net IO_H14_BANK15: now also U1.H14 (IO_L3N_T0_DQS_AD1N_15)
- net IO_J17_BANK15: now reaches J4.15 (Pin_15)
- net IO_J17_BANK15: now also U1.J17 (IO_L21N_T3_DQS_A18_15)
- net IO_H17_BANK15: now reaches J4.16 (Pin_16)
- net IO_H17_BANK15: now also U1.H17 (IO_L6P_T0_15)
- net IO_H15_BANK15: now reaches J4.17 (Pin_17)
- net IO_H15_BANK15: now also U1.H15 (IO_L5N_T0_AD9N_15)
- net IO_G15_BANK15: now reaches J4.18 (Pin_18)
- net IO_G15_BANK15: now also U1.G15 (IO_L2P_T0_AD8P_15)
- net IO_G16_BANK15: now reaches J4.19 (Pin_19)
- net IO_G16_BANK15: now also U1.G16 (IO_L2N_T0_AD8N_15)
- net IO_L16_BANK15: now reaches J4.2 (Pin_2)
- net IO_L16_BANK15: now also U1.L16 (IO_L23P_T3_~{FOE}_15)
- net IO_G17_BANK15: now reaches J4.20 (Pin_20)
- net IO_G17_BANK15: now also U1.G17 (IO_L4P_T0_15)
- net IO_G18_BANK15: now reaches J4.21 (Pin_21)
- net IO_G18_BANK15: now also U1.G18 (IO_L4N_T0_15)
- net IO_H18_BANK15: now reaches J4.22 (Pin_22)
- net IO_H18_BANK15: now also U1.H18 (IO_L6N_T0_VREF_15)
- net IO_H22_BANK15: now reaches J4.23 (Pin_23)
- net IO_H22_BANK15: now also U1.H22 (IO_L7N_T1_AD2N_15)
- net IO_H19_BANK15: now reaches J4.24 (Pin_24)
- net IO_H19_BANK15: now also U1.H19 (IO_L12N_T1_MRCC_15)
- net IO_J19_BANK15: now reaches J4.25 (Pin_25)
- net IO_J19_BANK15: now also U1.J19 (IO_L12P_T1_MRCC_15)
- net IO_J22_BANK15: now reaches J4.26 (Pin_26)
- net IO_J22_BANK15: now also U1.J22 (IO_L7P_T1_AD2P_15)
- net IO_J21_BANK15: now reaches J4.27 (Pin_27)
- net IO_J21_BANK15: now also U1.J21 (IO_L11N_T1_SRCC_15)
- net IO_J20_BANK15: now reaches J4.28 (Pin_28)
- net IO_J20_BANK15: now also U1.J20 (IO_L11P_T1_SRCC_15)
- net IO_K22_BANK15: now reaches J4.29 (Pin_29)
- net IO_K22_BANK15: now also U1.K22 (IO_L9N_T1_DQS_AD3N_15)
- net IO_M17_BANK15: now reaches J4.3 (Pin_3)
- net IO_M17_BANK15: now also U1.M17 (IO_25_15)
- net IO_K21_BANK15: now reaches J4.30 (Pin_30)
- net IO_K21_BANK15: now also U1.K21 (IO_L9P_T1_DQS_AD3P_15)
- net IO_L21_BANK15: now reaches J4.31 (Pin_31)
- net IO_L21_BANK15: now also U1.L21 (IO_L10N_T1_AD11N_15)
- net IO_L20_BANK15: now reaches J4.32 (Pin_32)
- net IO_L20_BANK15: now also U1.L20 (IO_L14N_T2_SRCC_15)
- net IO_M20_BANK15: now reaches J4.33 (Pin_33)
- net IO_M20_BANK15: now also U1.M20 (IO_L18N_T2_A23_15)
- net IO_M22_BANK15: now reaches J4.34 (Pin_34)
- net IO_M22_BANK15: now also U1.M22 (IO_L15N_T2_DQS_~{ADV}_15)
- net IO_M21_BANK15: now reaches J4.35 (Pin_35)
- net IO_M21_BANK15: now also U1.M21 (IO_L10P_T1_AD11P_15)
- net IO_N22_BANK15: now reaches J4.36 (Pin_36)
- net IO_N22_BANK15: now also U1.N22 (IO_L15P_T2_DQS_15)
- net IO_N20_BANK15: now reaches J4.37 (Pin_37)
- net IO_N20_BANK15: now also U1.N20 (IO_L18P_T2_A24_15)
- net IO_N19_BANK15: now reaches J4.38 (Pin_38)
- net IO_N19_BANK15: now also U1.N19 (IO_L17N_T2_A25_15)
- net IO_M18_BANK15: now reaches J4.39 (Pin_39)
- net IO_M18_BANK15: now also U1.M18 (IO_L16P_T2_A28_15)
- net IO_L18_BANK15: now reaches J4.4 (Pin_4)
- net IO_L18_BANK15: now also U1.L18 (IO_L16N_T2_A27_15)
- net IO_N18_BANK15: now reaches J4.40 (Pin_40)
- net IO_N18_BANK15: now also U1.N18 (IO_L17P_T2_A26_15)
- net IO_L15_BANK15: now reaches J4.5 (Pin_5)
- net IO_L15_BANK15: now also U1.L15 (IO_L22N_T3_A16_15)
- net IO_K16_BANK15: now reaches J4.6 (Pin_6)
- net IO_K16_BANK15: now also U1.K16 (IO_L23N_T3_~{FWE}_15)
- net IO_L19_BANK15: now reaches J4.7 (Pin_7)
- net IO_L19_BANK15: now also U1.L19 (IO_L14P_T2_SRCC_15)
- net IO_K19_BANK15: now reaches J4.8 (Pin_8)
- net IO_K19_BANK15: now also U1.K19 (IO_L13N_T2_MRCC_15)
- net IO_J15_BANK15: now reaches J4.9 (Pin_9)
- net IO_J15_BANK15: now also U1.J15 (IO_L5P_T0_AD9P_15)
- net IO_A13_BANK16: now reaches U1.A13 (IO_L10P_T1_16)
- net IO_A14_BANK16: now reaches U1.A14 (IO_L10N_T1_16)
- net IO_A14_BANK16: now also J3.17 (Pin_17)
- net IO_A15_BANK16: now reaches U1.A15 (IO_L9P_T1_DQS_16)
- net IO_A15_BANK16: now also J3.18 (Pin_18)
- net IO_A16_BANK16: now reaches U1.A16 (IO_L9N_T1_DQS_16)
- net IO_A16_BANK16: now also J3.22 (Pin_22)
- net IO_A18_BANK16: now reaches U1.A18 (IO_L17P_T2_16)
- net IO_A18_BANK16: now also J3.25 (Pin_25)
- net IO_A19_BANK16: now reaches U1.A19 (IO_L17N_T2_16)
- net IO_A19_BANK16: now also J3.28 (Pin_28)
- net IO_A20_BANK16: now reaches U1.A20 (IO_L16N_T2_16)
- net IO_A20_BANK16: now also J3.29 (Pin_29)
- net IO_A21_BANK16: now reaches U1.A21 (IO_L21N_T3_DQS_16)
- net IO_A21_BANK16: now also J3.30 (Pin_30)
- net IO_B13_BANK16: now reaches U1.B13 (IO_L8N_T1_16)
- net IO_B15_BANK16: now reaches U1.B15 (IO_L7P_T1_16)
- net IO_B15_BANK16: now also J3.14 (Pin_14)
- net IO_B16_BANK16: now reaches U1.B16 (IO_L7N_T1_16)
- net IO_B16_BANK16: now also J3.21 (Pin_21)
- net IO_B17_BANK16: now reaches U1.B17 (IO_L11P_T1_SRCC_16)
- net IO_B17_BANK16: now also J3.23 (Pin_23)
- net IO_B18_BANK16: now reaches U1.B18 (IO_L11N_T1_SRCC_16)
- net IO_B18_BANK16: now also J3.26 (Pin_26)
- net IO_B20_BANK16: now reaches U1.B20 (IO_L16P_T2_16)
- net IO_B20_BANK16: now also J3.31 (Pin_31)
- net IO_B21_BANK16: now reaches U1.B21 (IO_L21P_T3_DQS_16)
- net IO_B21_BANK16: now also J3.33 (Pin_33)
- net IO_B22_BANK16: now reaches U1.B22 (IO_L20N_T3_16)
- net IO_B22_BANK16: now also J3.32 (Pin_32)
- net IO_C13_BANK16: now reaches U1.C13 (IO_L8P_T1_16)
- net IO_C14_BANK16: now reaches U1.C14 (IO_L3P_T0_DQS_16)
- net IO_C15_BANK16: now reaches U1.C15 (IO_L3N_T0_DQS_16)
- net IO_C15_BANK16: now also J3.13 (Pin_13)
- net IO_C17_BANK16: now reaches U1.C17 (IO_L12N_T1_MRCC_16)
- net IO_C18_BANK16: now reaches U1.C18 (IO_L13P_T2_MRCC_16)
- net IO_C18_BANK16: now also J3.24 (Pin_24)
- net IO_C19_BANK16: now reaches U1.C19 (IO_L13N_T2_MRCC_16)
- net IO_C19_BANK16: now also J3.27 (Pin_27)
- net IO_C20_BANK16: now reaches U1.C20 (IO_L19N_T3_VREF_16)
- net IO_C20_BANK16: now also J3.35 (Pin_35)
- net IO_C22_BANK16: now reaches U1.C22 (IO_L20P_T3_16)
- net IO_C22_BANK16: now also J3.34 (Pin_34)
- net IO_D14_BANK16: now reaches U1.D14 (IO_L6P_T0_16)
- net IO_D15_BANK16: now reaches U1.D15 (IO_L6N_T0_VREF_16)
- net IO_D15_BANK16: now also J3.10 (Pin_10)
- net IO_D16_BANK16: now reaches U1.D16 (IO_L5N_T0_16)
- net IO_D16_BANK16: now also J3.9 (Pin_9)
- net IO_D17_BANK16: now reaches U1.D17 (IO_L12P_T1_MRCC_16)
- net IO_D17_BANK16: now also J3.20 (Pin_20)
- net IO_D19_BANK16: now reaches U1.D19 (IO_L14N_T2_SRCC_16)
- net IO_D19_BANK16: now also J3.12 (Pin_12)
- net IO_D20_BANK16: now reaches U1.D20 (IO_L19P_T3_16)
- net IO_D20_BANK16: now also J3.36 (Pin_36)
- net IO_D21_BANK16: now reaches U1.D21 (IO_L23N_T3_16)
- net IO_D21_BANK16: now also J3.38 (Pin_38)
- net IO_D22_BANK16: now reaches U1.D22 (IO_L22N_T3_16)
- net IO_D22_BANK16: now also J3.37 (Pin_37)
- net IO_E13_BANK16: now reaches U1.E13 (IO_L4P_T0_16)
- net IO_E14_BANK16: now reaches U1.E14 (IO_L4N_T0_16)
- net IO_E16_BANK16: now reaches U1.E16 (IO_L5P_T0_16)
- net IO_E16_BANK16: now also J3.2 (Pin_2)
- net IO_E17_BANK16: now reaches U1.E17 (IO_L2N_T0_16)
- net IO_E17_BANK16: now also J3.19 (Pin_19)
- net IO_E18_BANK16: now reaches U1.E18 (IO_L15N_T2_DQS_16)
- net IO_E18_BANK16: now also J3.16 (Pin_16)
- net IO_E19_BANK16: now reaches U1.E19 (IO_L14P_T2_SRCC_16)
- net IO_E19_BANK16: now also J3.11 (Pin_11)
- net IO_E21_BANK16: now reaches U1.E21 (IO_L23P_T3_16)
- net IO_E21_BANK16: now also J3.39 (Pin_39)
- net IO_E22_BANK16: now reaches U1.E22 (IO_L22P_T3_16)
- net IO_E22_BANK16: now also J3.40 (Pin_40)
- net IO_F13_BANK16: now reaches U1.F13 (IO_L1P_T0_16)
- net IO_F14_BANK16: now reaches U1.F14 (IO_L1N_T0_16)
- net IO_F14_BANK16: now also J3.6 (Pin_6)
- net IO_F15_BANK16: now reaches U1.F15 (IO_0_16)
- net IO_F15_BANK16: now also J3.5 (Pin_5)
- net IO_F16_BANK16: now reaches U1.F16 (IO_L2P_T0_16)
- net IO_F16_BANK16: now also J3.1 (Pin_1)
- net IO_F18_BANK16: now reaches U1.F18 (IO_L15P_T2_DQS_16)
- net IO_F18_BANK16: now also J3.15 (Pin_15)
- net IO_F19_BANK16: now reaches U1.F19 (IO_L18P_T2_16)
- net IO_F19_BANK16: now also J3.8 (Pin_8)
- net IO_F20_BANK16: now reaches U1.F20 (IO_L18N_T2_16)
- net IO_F20_BANK16: now also J3.7 (Pin_7)
- net IO_F21_BANK16: now reaches U1.F21 (IO_25_16)
- net IO_F21_BANK16: now also J3.4 (Pin_4)
- net IO_G21_BANK16: now reaches U1.G21 (IO_L24P_T3_16)
- net IO_G21_BANK16: now also J3.3 (Pin_3)
- net IO_G22_BANK16: now reaches U1.G22 (IO_L24N_T3_16)
- net IO_AA18_BANK14: now reaches U1.AA18 (IO_L17P_T2_A14_D30_14)
- net IO_AA18_BANK14: now also J5.39 (Pin_39)
- net IO_AA19_BANK14: now reaches U1.AA19 (IO_L15P_T2_DQS_~{RDWR}_14)
- net IO_AA19_BANK14: now also J5.38 (Pin_38)
- net IO_AA20_BANK14: now reaches U1.AA20 (IO_L8P_T1_D11_14)
- net IO_AA20_BANK14: now also J5.33 (Pin_33)
- net IO_AA21_BANK14: now reaches U1.AA21 (IO_L8N_T1_D12_14)
- net IO_AA21_BANK14: now also J5.34 (Pin_34)
- net IO_AB18_BANK14: now reaches U1.AB18 (IO_L17N_T2_A13_D29_14)
- net IO_AB18_BANK14: now also J5.40 (Pin_40)
- net IO_AB20_BANK14: now reaches U1.AB20 (IO_L15N_T2_DQS_DOUT_~{CSO}_14)
- net IO_AB20_BANK14: now also J5.35 (Pin_35)
- net IO_AB21_BANK14: now reaches U1.AB21 (IO_L10P_T1_D14_14)
- net IO_AB21_BANK14: now also J5.36 (Pin_36)
- net IO_AB22_BANK14: now reaches U1.AB22 (IO_L10N_T1_D15_14)
- net IO_AB22_BANK14: now also J5.37 (Pin_37)
- net IO_N13_BANK14: now reaches U1.N13 (IO_L23P_T3_A03_D19_14)
- net IO_N14_BANK14: now reaches U1.N14 (IO_L23N_T3_A02_D18_14)
- net IO_N15_BANK14: now reaches U1.N15 (IO_25_14)
- net IO_N17_BANK14: now reaches U1.N17 (IO_L21P_T3_DQS_14)
- net IO_N17_BANK14: now also J5.12 (Pin_12)
- net IO_P14_BANK14: now reaches U1.P14 (IO_L19P_T3_A10_D26_14)
- net IO_P15_BANK14: now reaches U1.P15 (IO_L22P_T3_A05_D21_14)
- net IO_P15_BANK14: now also J5.3 (Pin_3)
- net IO_P16_BANK14: now reaches U1.P16 (IO_L24P_T3_A01_D17_14)
- net IO_P16_BANK14: now also J5.4 (Pin_4)
- net IO_P17_BANK14: now reaches U1.P17 (IO_L21N_T3_DQS_A06_D22_14)
- net IO_P17_BANK14: now also J5.11 (Pin_11)
- net IO_P19_BANK14: now reaches U1.P19 (IO_L5P_T0_D06_14)
- net IO_P19_BANK14: now also J5.19 (Pin_19)
- net IO_P20_BANK14: now reaches U1.P20 (IO_0_14)
- net IO_P20_BANK14: now also J5.20 (Pin_20)
- net IO_R14_BANK14: now reaches U1.R14 (IO_L19N_T3_A09_D25_VREF_14)
- net IO_R16_BANK14: now reaches U1.R16 (IO_L22N_T3_A04_D20_14)
- net IO_R16_BANK14: now also J5.7 (Pin_7)
- net IO_R17_BANK14: now reaches U1.R17 (IO_L24N_T3_A00_D16_14)
- net IO_R17_BANK14: now also J5.8 (Pin_8)
- net IO_R18_BANK14: now reaches U1.R18 (IO_L20P_T3_A08_D24_14)
- net IO_R18_BANK14: now also J5.15 (Pin_15)
- net IO_R19_BANK14: now reaches U1.R19 (IO_L5N_T0_D07_14)
- net IO_R19_BANK14: now also J5.16 (Pin_16)
- net IO_T18_BANK14: now reaches U1.T18 (IO_L20N_T3_A07_D23_14)
- net IO_T18_BANK14: now also J5.17 (Pin_17)
- net IO_T20_BANK14: now reaches U1.T20 (IO_L6N_T0_D08_VREF_14)
- net IO_T20_BANK14: now also J5.18 (Pin_18)
- net IO_T21_BANK14: now reaches U1.T21 (IO_L4P_T0_D04_14)
- net IO_T21_BANK14: now also J5.21 (Pin_21)
- net IO_U17_BANK14: now reaches U1.U17 (IO_L18P_T2_A12_D28_14)
- net IO_U17_BANK14: now also J5.14 (Pin_14)
- net IO_U18_BANK14: now reaches U1.U18 (IO_L18N_T2_A11_D27_14)
- net IO_U18_BANK14: now also J5.13 (Pin_13)
- net IO_U20_BANK14: now reaches U1.U20 (IO_L11P_T1_SRCC_14)
- net IO_U20_BANK14: now also J5.24 (Pin_24)
- net IO_U21_BANK14: now reaches U1.U21 (IO_L4N_T0_D05_14)
- net IO_U21_BANK14: now also J5.22 (Pin_22)
- net IO_U22_BANK14: now reaches U1.U22 (IO_L3P_T0_DQS_~{PUDC}_14)
- net IO_U22_BANK14: now also J5.23 (Pin_23)
- net IO_V17_BANK14: now reaches U1.V17 (IO_L16P_T2_~{CSI}_14)
- net IO_V17_BANK14: now also J5.9 (Pin_9)
- net IO_V18_BANK14: now reaches U1.V18 (IO_L14P_T2_SRCC_14)
- net IO_V18_BANK14: now also J5.10 (Pin_10)
- net IO_V19_BANK14: now reaches U1.V19 (IO_L14N_T2_SRCC_14)
- net IO_V19_BANK14: now also J5.27 (Pin_27)
- net IO_V20_BANK14: now reaches U1.V20 (IO_L11N_T1_SRCC_14)
- net IO_V20_BANK14: now also J5.25 (Pin_25)
- net IO_V22_BANK14: now reaches U1.V22 (IO_L3N_T0_DQS_EMCCLK_14)
- net IO_V22_BANK14: now also J5.26 (Pin_26)
- net IO_W17_BANK14: now reaches U1.W17 (IO_L16N_T2_A15_D31_14)
- net IO_W17_BANK14: now also J5.6 (Pin_6)
- net IO_W19_BANK14: now reaches U1.W19 (IO_L12P_T1_MRCC_14)
- net IO_W19_BANK14: now also J5.28 (Pin_28)
- net IO_W20_BANK14: now reaches U1.W20 (IO_L12N_T1_MRCC_14)
- net IO_W20_BANK14: now also J5.5 (Pin_5)
- net IO_W21_BANK14: now reaches U1.W21 (IO_L7P_T1_D09_14)
- net IO_W21_BANK14: now also J5.30 (Pin_30)
- net IO_W22_BANK14: now reaches U1.W22 (IO_L7N_T1_D10_14)
- net IO_W22_BANK14: now also J5.29 (Pin_29)
- net IO_Y18_BANK14: now reaches U1.Y18 (IO_L13P_T2_MRCC_14)
- net IO_Y18_BANK14: now also J5.1 (Pin_1)
- net IO_Y19_BANK14: now reaches U1.Y19 (IO_L13N_T2_MRCC_14)
- net IO_Y19_BANK14: now also J5.2 (Pin_2)
- net IO_Y21_BANK14: now reaches U1.Y21 (IO_L9P_T1_DQS_14)
- net IO_Y21_BANK14: now also J5.31 (Pin_31)
- net IO_Y22_BANK14: now reaches U1.Y22 (IO_L9N_T1_DQS_D13_14)
- net IO_Y22_BANK14: now also J5.32 (Pin_32)
- net IO_G13_BANK15: now reaches U1.G13 (IO_L1N_T0_AD0N_15)
- net IO_G20_BANK15: now reaches U1.G20 (IO_L8N_T1_AD10N_15)
- net IO_H13_BANK15: now reaches U1.H13 (IO_L1P_T0_AD0P_15)
- net IO_H20_BANK15: now reaches U1.H20 (IO_L8P_T1_AD10P_15)
- net IO_K13_BANK15: now reaches U1.K13 (IO_L19P_T3_A22_15)
- net IO_K14_BANK15: now reaches U1.K14 (IO_L19N_T3_A21_VREF_15)
- net IO_L13_BANK15: now reaches U1.L13 (IO_L20N_T3_A19_15)
- net IO_L14_BANK15: now reaches U1.L14 (IO_L22P_T3_A17_15)
- net IO_M13_BANK15: now reaches U1.M13 (IO_L20P_T3_A20_15)
- net IO_M15_BANK15: now reaches U1.M15 (IO_L24P_T3_RS1_15)
- net M0 renamed M2_BANK0
- net M1 renamed M1_BANK0
- net M2 renamed M0_BANK0
- net QPI_CCLK renamed QPI_CCLK_BANK0
- net QPI_CS renamed QPI_CS_BANK14
- net QPI_D0 renamed QPI_D0_BANK14
- net QPI_D1 renamed QPI_D1_BANK14
- net QPI_D2 renamed QPI_D2_BANK14
- net QPI_D3 renamed QPI_D3_BANK14
Other:
- moved on the sheet: C33, C53, C54, C55, C56, J3, J4, J5, J6, U1A, U1B, U1C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

Commit message: idk
Parts:
- added TP3, TP4, TP5, TP6, TP7, TP8: TestPoint, TestPoint:TestPoint_Pad_D1.0mm, symbol Connector:TestPoint
- U1: LCSC part number (none) -> C1521841; automotive No -> (none); category IC -> (none); device class L1 Integrated Circuits (ICs) -> (none); device class L2 Embedded Processors and Controllers -> (none); device class L3 FPGAs - Field Programmable Gate Arrays -> (none); digikey description IC FPGA ARTIX7 285 I/O 484FCBGA -> (none); lead free Yes -> (none); max supply voltage 3.465V -> (none); min supply voltage 0.95V -> (none); number of I/Os 285 -> (none); number of logic blocks 33650 -> (none); number of logic elements cells 215360 -> (none); package FBG484 -> (none); release date 1402480027 -> (none); rohs Yes -> (none); speed grade 3 -> (none); standoff height 0.4mm -> (none); temperature range high +100°C -> (none); temperature range low 0°C -> (none); vault revision 8A58598F-56A5-4DEC-BA3F-FDB4B6026E25 -> (none)
Connections:
- net DONE is gone; now on net DONE_BANK0: U1.G11 (DONE_0)
- net +3V3: no longer C33.1, U1.U8 (CFGBVS_0)
- net DDR3/~{DDR_RST}: now also U1.Y1 (IO_L5N_T0_34)
- net GND: now also J7.1 (Pin_1), J7.12 (Pin_12), J7.14 (Pin_14), J7.16 (Pin_16), J7.18 (Pin_18), J7.20 (Pin_20), J7.21 (Pin_21), J7.23 (Pin_23), J7.25 (Pin_25), J7.27 (Pin_27), J7.29 (Pin_29), J7.40 (Pin_40), TP3.1
- net M0_BANK0: now also J7.3 (Pin_3)
- net M1_BANK0: now also J7.6 (Pin_6)
- net M2_BANK0: now also J7.7 (Pin_7)
- net MTGAVTT: now also TP8.1
- net QPI_CCLK_BANK0: now also J7.39 (Pin_39)
- net QPI_CS_BANK14: now also J7.38 (Pin_38)
- net QPI_D0_BANK14: now also J7.34 (Pin_34)
- net QPI_D1_BANK14: now also J7.35 (Pin_35)
- net QPI_D2_BANK14: now also J7.36 (Pin_36)
- net QPI_D3_BANK14: now also J7.37 (Pin_37)
- net TCK_BANK0: now also J7.32 (Pin_32)
- net TDI_BANK0: now also J7.31 (Pin_31)
- net TDO_BANK0: now also J7.30 (Pin_30)
- net TMS_BANK0: now also J7.33 (Pin_33)
- net ~{PROG}_BANK0: now reaches U1.N12 (~{PROGRAM}_0)
- net ~{PROG}_BANK0: now also J7.4 (Pin_4)
- net ~{INIT}_BANK0: now reaches U1.U12 (~{INIT}_0)
- net ~{INIT}_BANK0: now also J7.5 (Pin_5)
- net VBANK14: now reaches J7.13 (Pin_13)
- net VBANK14: now also C33.1, J7.28 (Pin_28), U1.U8 (CFGBVS_0)
- net VBANK13: now reaches J7.15 (Pin_15)
- net VBANK13: now also J7.26 (Pin_26)
- net VBANK15: now reaches J7.17 (Pin_17)
- net VBANK15: now also J7.24 (Pin_24)
- net VBANK16: now reaches J7.19 (Pin_19)
- net VBANK16: now also J7.22 (Pin_22)
- net DONE_BANK0: now reaches J7.2 (Pin_2)
- net IO_A13_BANK16: no longer names the net of U1.A13 (IO_L10P_T1_16)
- net IO_B13_BANK16: no longer names the net of U1.B13 (IO_L8N_T1_16)
- net IO_C13_BANK16: no longer names the net of U1.C13 (IO_L8P_T1_16)
- net IO_C14_BANK16: no longer names the net of U1.C14 (IO_L3P_T0_DQS_16)
- net IO_C17_BANK16: no longer names the net of U1.C17 (IO_L12N_T1_MRCC_16)
- net IO_D14_BANK16: no longer names the net of U1.D14 (IO_L6P_T0_16)
- net IO_E13_BANK16: no longer names the net of U1.E13 (IO_L4P_T0_16)
- net IO_E14_BANK16: no longer names the net of U1.E14 (IO_L4N_T0_16)
- net IO_F13_BANK16: no longer names the net of U1.F13 (IO_L1P_T0_16)
- net IO_G13_BANK15: no longer names the net of U1.G13 (IO_L1N_T0_AD0N_15)
- net IO_G20_BANK15: no longer names the net of U1.G20 (IO_L8N_T1_AD10N_15)
- net IO_G22_BANK16: no longer names the net of U1.G22 (IO_L24N_T3_16)
- net IO_H13_BANK15: no longer names the net of U1.H13 (IO_L1P_T0_AD0P_15)
- net IO_H20_BANK15: no longer names the net of U1.H20 (IO_L8P_T1_AD10P_15)
- net IO_K13_BANK15: no longer names the net of U1.K13 (IO_L19P_T3_A22_15)
- net IO_K14_BANK15: no longer names the net of U1.K14 (IO_L19N_T3_A21_VREF_15)
- net IO_L13_BANK15: no longer names the net of U1.L13 (IO_L20N_T3_A19_15)
- net IO_L14_BANK15: no longer names the net of U1.L14 (IO_L22P_T3_A17_15)
- net IO_M13_BANK15: no longer names the net of U1.M13 (IO_L20P_T3_A20_15)
- net IO_M15_BANK15: no longer names the net of U1.M15 (IO_L24P_T3_RS1_15)
- net IO_N13_BANK14: no longer names the net of U1.N13 (IO_L23P_T3_A03_D19_14)
- net IO_N14_BANK14: no longer names the net of U1.N14 (IO_L23N_T3_A02_D18_14)
- net IO_N15_BANK14: no longer names the net of U1.N15 (IO_25_14)
- net IO_P14_BANK14: no longer names the net of U1.P14 (IO_L19P_T3_A10_D26_14)
- net IO_R14_BANK14: no longer names the net of U1.R14 (IO_L19N_T3_A09_D25_VREF_14)
- new net +1V0: TP6.1
- new net +1V35: TP4.1
- new net +1V8: TP5.1
- new net MTGAVCC: TP7.1
- no-connect marks 0 -> 61
Other:
- sheet Power ports: added none; removed P_{GOOD}
- note removed: "resv"
- moved on the sheet: C33, J7
