File: carrier-basic/carrier-basic.kicad_pcb (KiCad board)
At the start: 4 copper layers, 150 x 150 mm, 21 parts, among them J1 Conn_02x20_Counter_Clockwise, J10 Conn_02x06_Odd_Even, J11 Conn_02x06_Odd_Even, J12 Conn_02x06_Odd_Even, J13 Conn_02x06_Odd_Even, J2 Conn_02x20_Counter_Clockwise, J3 Conn_02x20_Counter_Clockwise, J4 Conn_02x20_Counter_Clockwise, J5 Conn_02x20_Counter_Clockwise, J6 Conn_02x20_Counter_Clockwise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

Commit message: Some more work on the carrier
Parts:
- added H5: MountingHole_Pad, MountingHole:MountingHole_4mm_Pad, F.Cu at (169.0, 31.0)
- added H6: MountingHole_Pad, MountingHole:MountingHole_4mm_Pad, F.Cu at (31.0, 31.0)
- added H7: MountingHole_Pad, MountingHole:MountingHole_4mm_Pad, F.Cu at (169.0, 169.0)
- added H8: MountingHole_Pad, MountingHole:MountingHole_4mm_Pad, F.Cu at (31.0, 169.0)
- moved J13 254.0 mm to (-91.4, 134.6)
- moved J12 24.1 mm to (161.3, 157.2)
- moved J11 16.5 mm to (161.3, 131.8)
- moved J10 8.92 mm to (161.3, 106.3)
- moved J8 6.39 mm to (161.3, 55.5)
- moved DSub1 6.19 mm to (138.0, 42.9)
- moved J9 1.46 mm to (161.3, 81.0)
Routing:
- net unconnected-(J10-Pin_11-Pad11): track 2.04 -> 0.00 mm
Other:
- outline, holes or cut-outs redrawn
